Commit message: 1202 수정

File: src/assets/urdf/franka_panda/franka_panda_handle/model.urdf (robot description, URDF)
Before this commit: robot panda, 13 links, 12 joints
Links:
- link panda_stick: geometry collision cylinder length=0.04 radius=0.01; visual cylinder length=0.0065 radius=0.022

File: src/assets/urdf/franka_panda/franka_panda_handle/project_hole.urdf (robot description, URDF)
Before this commit: robot project_hole, 1 links, 0 joints
Links:
- link base_link: mass 0.053575148377838 -> 0.0535751483778379
